Commit message: Fix: Possible fix to solve the simulation LiDAR  URDF bug

File: software/src/omnicare_description/urdf/robot.xacro (robot description, xacro)
@@ -6,13 +6,14 @@
     </xacro:if>
     <xacro:unless value="$(arg sim_mode)">
+        <!-- To fix the LiDAR Link bug between real robot URDF and sim robot  -->
+        <link name="lidar_link"></link>
+        <joint name="lidar_to_base" type="fixed">
+            <parent link="base_link" />
+            <child link="lidar_link" />
+            <origin rpy="0.0 0 3.14" xyz="0 0 0" />
+        </joint>
         <xacro:include filename="$(find omnicare_description)/urdf/ros2_control.xacro" />
     </xacro:unless>
     <xacro:include filename="$(find omnicare_description)/urdf/camera.xacro"/>
-    <link name="lidar_link"></link>
-    <joint name="lidar_to_base" type="fixed">
-        <parent link="base_link" />
-        <child link="lidar_link" />
-        <origin rpy="0.0 0 3.14" xyz="0 0 0" />
-    </joint>
     <joint name="base_footprint_to_base_link" type="fixed">
         <parent link="base_footprint" />

Commit message: Update: Fixed OmniCare sliding in Gazebo

File: software/src/omnicare_description/urdf/robot.xacro (robot description, xacro)
@@ -15,5 +15,5 @@
         <xacro:include filename="$(find omnicare_description)/urdf/ros2_control.xacro" />
     </xacro:unless>
-    <xacro:include filename="$(find omnicare_description)/urdf/camera.xacro"/>
+    <xacro:include filename="$(find omnicare_description)/urdf/camera.xacro" />
     <joint name="base_footprint_to_base_link" type="fixed">
         <parent link="base_footprint" />
@@ -316,12 +316,13 @@
         </inertial>
     </link>
-    <joint name="w1_external_1_passive" type="continuous">
+    <joint name="w1_external_1_passive" type="fixed">
         <origin xyz="0.01750000000000022024 -0.050000000000000002776 -0.046999999999999930722"
             rpy="-3.141592653589793116 -1.570796326794896558 0" />
         <parent link="roda" />
         <child link="rolete" />
-        <axis xyz="0 0 1" />
-        <limit effort="1" velocity="20" />
-        <joint_properties friction="0.0" />
+        <axis xyz="0 0 1">
+            <dynamics damping="1.0" friction="1.0" /> <!-- ISSO FUNCIONA -->
+        </axis>
+        <limit effort="1" velocity="20" />
     </joint>
     <link name="rolete_2">
@@ -354,12 +355,13 @@
         </inertial>
     </link>
-    <joint name="w1_external_2_passive" type="continuous">
+    <joint name="w1_external_2_passive" type="fixed">
         <origin xyz="0.052051270189221954254 -0.009844555433772231301 -0.047000000000000041744"
             rpy="1.570796326794896558 4.1633363423452281929e-17 2.6179938779914921909" />
         <parent link="roda" />
         <child link="rolete_2" />
-        <axis xyz="0 0 1" />
-        <limit effort="1" velocity="20" />
-        <joint_properties friction="0.0" />
+        <axis xyz="0 0 1">
+            <dynamics damping="1.0" friction="1.0" /> <!-- ISSO FUNCIONA -->
+        </axis>
+        <limit effort="1" velocity="20" />
     </joint>
     <link name="rolete_3">
@@ -392,12 +394,13 @@
         </inertial>
     </link>
-    <joint name="w1_external_3_passive" type="continuous">
+    <joint name="w1_external_3_passive" type="fixed">
         <origin xyz="0.052051270189221968132 0.0098445554337722868121 -0.047000000000000041744"
             rpy="-1.570796326794896558 4.163336342345265787e-17 -2.6179938779914921909" />
         <parent link="roda" />
         <child link="rolete_3" />
-        <axis xyz="0 0 1" />
-        <limit effort="1" velocity="20" />
-        <joint_properties friction="0.0" />
+        <axis xyz="0 0 1">
+            <dynamics damping="1.0" friction="1.0" /> <!-- ISSO FUNCIONA -->
+        </axis>
+        <limit effort="1" velocity="20" />
     </joint>
     <link name="rolete_4">
@@ -429,12 +432,13 @@
         </inertial>
     </link>
-    <joint name="w1_external_4_passive" type="continuous">
+    <joint name="w1_external_4_passive" type="fixed">
         <origin xyz="0.01750000000000022024 0.050000000000000002776 -0.046999999999999930722"
             rpy="-3.141592653589793116 -1.570796326794896558 0" />
         <parent link="roda" />
         <child link="rolete_4" />
-        <axis xyz="0 0 1" />
-        <limit effort="1" velocity="20" />
-        <joint_properties friction="0.0" />
+        <axis xyz="0 0 1">
+            <dynamics damping="1.0" friction="1.0" /> <!-- ISSO FUNCIONA -->
+        </axis>
+        <limit effort="1" velocity="20" />
     </joint>
     <link name="rolete_5">
@@ -469,12 +473,13 @@
         </inertial>
     </link>
-    <joint name="w1_external_5_passive" type="continuous">
+    <joint name="w1_external_5_passive" type="fixed">
         <origin xyz="-0.034551270189221897078 0.040155444566227743719 -0.046999999999999930722"
             rpy="1.570796326794896558 9.7144514654709209156e-17 2.6179938779914921909" />
         <parent link="roda" />
         <child link="rolete_5" />
-        <axis xyz="0 0 1" />
-        <limit effort="1" velocity="20" />
-        <joint_properties friction="0.0" />
+        <axis xyz="0 0 1">
+            <dynamics damping="1.0" friction="1.0" /> <!-- ISSO FUNCIONA -->
+        </axis>
+        <limit effort="1" velocity="20" />
     </joint>
     <link name="rolete_6">
@@ -507,12 +512,13 @@
         </inertial>
     </link>
-    <joint name="w1_external_6_passive" type="continuous">
+    <joint name="w1_external_6_passive" type="fixed">
         <origin xyz="-0.034551270189221897078 -0.040155444566227743719 -0.046999999999999986233"
             rpy="-1.570796326794896558 4.163336342345242984e-17 -2.6179938779914930791" />
         <parent link="roda" />
         <child link="rolete_6" />
-        <axis xyz="0 0 1" />
-        <limit effort="1" velocity="20" />
-        <joint_properties friction="0.0" />
+        <axis xyz="0 0 1">
+            <dynamics damping="1.0" friction="1.0" /> <!-- ISSO FUNCIONA -->
+        </axis>
+        <limit effort="1" velocity="20" />
     </joint>
     <link name="rolete_7">
@@ -547,12 +553,13 @@
         </inertial>
     </link>
-    <joint name="w1_internal_1_passive" type="continuous">
+    <joint name="w1_internal_1_passive" type="fixed">
         <origin xyz="0.0098445554337722885468 -0.052051270189221947315 -0.02899999999999994249"
             rpy="0.52359877559829937077 -1.570796326794896558 0" />
         <parent link="roda" />
         <child link="rolete_7" />
-        <axis xyz="0 0 1" />
-        <limit effort="1" velocity="20" />
-        <joint_properties friction="0.0" />
+        <axis xyz="0 0 1">
+            <dynamics damping="1.0" friction="1.0" /> <!-- ISSO FUNCIONA -->
+        </axis>
+        <limit effort="1" velocity="20" />
     </joint>
     <link name="rolete_8">
@@ -586,12 +593,13 @@
         </inertial>
     </link>
-    <joint name="w1_internal_2_passive" type="continuous">
+    <joint name="w1_internal_2_passive" type="fixed">
         <origin xyz="0.050000000000000016653 -0.017500000000000019013 -0.028999999999999970246"
             rpy="-1.570796326794896558 1.035468818874435832e-17 3.141592653589793116" />
         <parent link="roda" />
         <child link="rolete_8" />
-        <axis xyz="0 0 1" />
-        <limit effort="1" velocity="20" />
-        <joint_properties friction="0.0" />
+        <axis xyz="0 0 1">
+            <dynamics damping="1.0" friction="1.0" /> <!-- ISSO FUNCIONA -->
+        </axis>
+        <limit effort="1" velocity="20" />
     </joint>
     <link name="rolete_9">
@@ -624,12 +632,13 @@
         </inertial>
     </link>
-    <joint name="w1_internal_3_passive" type="continuous">
+    <joint name="w1_internal_3_passive" type="fixed">
         <origin xyz="0.0098445554337722469135 0.052051270189221926499 -0.028999999999999998002"
             rpy="-0.5235987755982990377 -1.570796326794896558 0" />
         <parent link="roda" />
         <child link="rolete_9" />
-        <axis xyz="0 0 1" />
-        <limit effort="1" velocity="20" />
-        <joint_properties friction="0.0" />
+        <axis xyz="0 0 1">
+            <dynamics damping="1.0" friction="1.0" /> <!-- ISSO FUNCIONA -->
+        </axis>
+        <limit effort="1" velocity="20" />
     </joint>
     <link name="rolete_10">
@@ -664,12 +673,13 @@
         </inertial>
     </link>
-    <joint name="w1_internal_4_passive" type="continuous">
+    <joint name="w1_internal_4_passive" type="fixed">
         <origin xyz="-0.0098445554337722486482 0.052051270189221954254 -0.028999999999999970246"
             rpy="-2.6179938779914890823 -1.570796326794896558 0" />
         <parent link="roda" />
         <child link="rolete_10" />
-        <axis xyz="0 0 1" />
-        <limit effort="1" velocity="20" />
-        <joint_properties friction="0.0" />
+        <axis xyz="0 0 1">
+            <dynamics damping="1.0" friction="1.0" /> <!-- ISSO FUNCIONA -->
+        </axis>
+        <limit effort="1" velocity="20" />
     </joint>
     <link name="rolete_11">
@@ -702,12 +712,13 @@
         </inertial>
     </link>
-    <joint name="w1_internal_5_passive" type="continuous">
+    <joint name="w1_internal_5_passive" type="fixed">
         <origin xyz="-0.049999999999999988898 -0.017500000000000001665 -0.028999999999999970246"
             rpy="-1.570796326794896558 6.5865839420001391858e-17 -3.1415926535897926719" />
         <parent link="roda" />
         <child link="rolete_11" />
-        <axis xyz="0 0 1" />
-        <limit effort="1" velocity="20" />
-        <joint_properties friction="0.0" />
+        <axis xyz="0 0 1">
+            <dynamics damping="1.0" friction="1.0" /> <!-- ISSO FUNCIONA -->
+        </axis>
+        <limit effort="1" velocity="20" />
     </joint>
     <link name="rolete_12">
@@ -742,12 +753,13 @@
         </inertial>
     </link>
-    <joint name="w1_internal_6_passive" type="continuous">
+    <joint name="w1_internal_6_passive" type="fixed">
         <origin xyz="-0.0098445554337722746691 -0.052051270189221933438 -0.028999999999999998002"
             rpy="2.6179938779914944114 -1.570796326794896558 0" />
         <parent link="roda" />
         <child link="rolete_12" />
-        <axis xyz="0 0 1" />
-        <limit effort="1" velocity="20" />
-        <joint_properties friction="0.0" />
+        <axis xyz="0 0 1">
+            <dynamics damping="1.0" friction="1.0" /> <!-- ISSO FUNCIONA -->
+        </axis>
+        <limit effort="1" velocity="20" />
     </joint>
     <joint name="wheel1_speed" type="continuous">
@@ -756,7 +768,8 @@
         <parent link="base" />
         <child link="roda" />
-        <axis xyz="0 0 1" />
-        <limit effort="1" velocity="20" />
-        <joint_properties friction="0.1" />
+        <axis xyz="0 0 1">
+            <dynamics damping="0.1" friction="0.2" /> <!-- ISSO FUNCIONA -->
+        </axis>
+        <limit effort="1" velocity="200" />
     </joint>
     <link name="roda_2">
@@ -816,12 +829,13 @@
         </inertial>
     </link>
-    <joint name="w2_external_1_passive" type="continuous">
+    <joint name="w2_external_1_passive" type="fixed">
         <origin xyz="0.017500000000000001665 -0.050000000000000002776 -0.046999999999999986233"
             rpy="-3.141592653589793116 -1.570796326794896558 0" />
         <parent link="roda_2" />
         <child link="rolete_13" />
-        <axis xyz="0 0 1" />
-        <limit effort="1" velocity="20" />
-        <joint_properties friction="0.0" />
+        <axis xyz="0 0 1">
+            <dynamics damping="1.0" friction="1.0" /> <!-- ISSO FUNCIONA -->
+        </axis>
+        <limit effort="1" velocity="20" />
     </joint>
     <link name="rolete_14">
@@ -856,12 +870,13 @@
         </inertial>
     </link>
-    <joint name="w2_external_2_passive" type="continuous">
+    <joint name="w2_external_2_passive" type="fixed">
         <origin xyz="0.052051270189221961193 -0.0098445554337722798732 -0.046999999999999986233"
             rpy="-1.570796326794896558 8.3266726846886740532e-17 -0.52359877559829937077" />
         <parent link="roda_2" />
         <child link="rolete_14" />
-        <axis xyz="0 0 1" />
-        <limit effort="1" velocity="20" />
-        <joint_properties friction="0.0" />
+        <axis xyz="0 0 1">
+            <dynamics damping="1.0" friction="1.0" /> <!-- ISSO FUNCIONA -->
+        </axis>
+        <limit effort="1" velocity="20" />
     </joint>
     <link name="rolete_15">
@@ -894,12 +909,13 @@
         </inertial>
     </link>
-    <joint name="w2_external_3_passive" type="continuous">
+    <joint name="w2_external_3_passive" type="fixed">
         <origin xyz="0.0345512701892218832 0.04015544456622767433 -0.046999999999999986233"
             rpy="-1.570796326794896558 -1.9428902930940232062e-16 0.5235987755982980385" />
         <parent link="roda_2" />
         <child link="rolete_15" />
-        <axis xyz="0 0 1" />
-        <limit effort="1" velocity="20" />
-        <joint_properties friction="0.0" />
+        <axis xyz="0 0 1">
+            <dynamics damping="1.0" friction="1.0" /> <!-- ISSO FUNCIONA -->
+        </axis>
+        <limit effort="1" velocity="20" />
     </joint>
     <link name="rolete_16">
@@ -931,12 +947,13 @@
         </inertial>
     </link>
-    <joint name="w2_external_4_passive" type="continuous">
+    <joint name="w2_external_4_passive" type="fixed">
         <origin xyz="0.017500000000000001665 0.050000000000000002776 -0.046999999999999986233"
             rpy="-3.141592653589793116 -1.570796326794896558 0" />
         <parent link="roda_2" />
         <child link="rolete_16" />
-        <axis xyz="0 0 1" />
-        <limit effort="1" velocity="20" />
-        <joint_properties friction="0.0" />
+        <axis xyz="0 0 1">
+            <dynamics damping="1.0" friction="1.0" /> <!-- ISSO FUNCIONA -->
+        </axis>
+        <limit effort="1" velocity="20" />
     </joint>
     <link name="rolete_17">
@@ -969,12 +986,13 @@
         </inertial>
     </link>
-    <joint name="w2_external_5_passive" type="continuous">
+    <joint name="w2_external_5_passive" type="fixed">
         <origin xyz="-0.034551270189221931772 0.040155444566227688208 -0.047000000000000041744"
             rpy="-1.570796326794896558 2.7755575615628950488e-17 -0.5235987755982990377" />
         <parent link="roda_2" />
         <child link="rolete_17" />
-        <axis xyz="0 0 1" />
-        <limit effort="1" velocity="20" />
-        <joint_properties friction="0.0" />
+        <axis xyz="0 0 1">
+            <dynamics damping="1.0" friction="1.0" /> <!-- ISSO FUNCIONA -->
+        </axis>
+        <limit effort="1" velocity="20" />
     </joint>
     <link name="rolete_18">
@@ -1007,12 +1025,13 @@
         </inertial>
     </link>
-    <joint name="w2_external_6_passive" type="continuous">
+    <joint name="w2_external_6_passive" type="fixed">
         <origin xyz="-0.052051270189221968132 -0.0098445554337723215066 -0.046999999999999986233"
             rpy="-1.570796326794896558 -2.4980018054065997508e-16 0.52359877559829848259" />
         <parent link="roda_2" />
         <child link="rolete_18" />
-        <axis xyz="0 0 1" />
-        <limit effort="1" velocity="20" />
-        <joint_properties friction="0.0" />
+        <axis xyz="0 0 1">
+            <dynamics damping="1.0" friction="1.0" /> <!-- ISSO FUNCIONA -->
+        </axis>
+        <limit effort="1" velocity="20" />
     </joint>
     <link name="rolete_19">
@@ -1045,12 +1064,13 @@
         </inertial>
     </link>
-    <joint name="w2_internal_1_passive" type="continuous">
+    <joint name="w2_internal_1_passive" type="fixed">
         <origin xyz="0.0098445554337722798732 -0.052051270189221954254 -0.028999999999999998002"
             rpy="0.52359877559829937077 -1.570796326794896558 0" />
         <parent link="roda_2" />
         <child link="rolete_19" />
-        <axis xyz="0 0 1" />
-        <limit effort="1" velocity="20" />
-        <joint_properties friction="0.0" />
+        <axis xyz="0 0 1">
+            <dynamics damping="1.0" friction="1.0" /> <!-- ISSO FUNCIONA -->
+        </axis>
+        <limit effort="1" velocity="20" />
     </joint>
     <link name="rolete_20">
@@ -1084,12 +1104,13 @@
         </inertial>
     </link>
-    <joint name="w2_internal_2_passive" type="continuous">
+    <joint name="w2_internal_2_passive" type="fixed">
         <origin xyz="0.050000000000000030531 0.017500000000000015543 -0.029000000000000025757"
             rpy="-1.570796326794896558 1.0888646801245511308e-17 0" />
         <parent link="roda_2" />
         <child link="rolete_20" />
-        <axis xyz="0 0 1" />
-        <limit effort="1" velocity="20" />
-        <joint_properties friction="0.0" />
+        <axis xyz="0 0 1">
+            <dynamics damping="1.0" friction="1.0" /> <!-- ISSO FUNCIONA -->
+        </axis>
+        <limit effort="1" velocity="20" />
     </joint>
     <link name="rolete_21">
@@ -1122,12 +1143,13 @@
         </inertial>
     </link>
-    <joint name="w2_internal_3_passive" type="continuous">
+    <joint name="w2_internal_3_passive" type="fixed">
         <origin xyz="0.0098445554337723163024 0.052051270189221954254 -0.028999999999999970246"
             rpy="-0.52359877559829870464 -1.570796326794896558 0" />
         <parent link="roda_2" />
         <child link="rolete_21" />
-        <axis xyz="0 0 1" />
-        <limit effort="1" velocity="20" />
-        <joint_properties friction="0.0" />
+        <axis xyz="0 0 1">
+            <dynamics damping="1.0" friction="1.0" /> <!-- ISSO FUNCIONA -->
+        </axis>
+        <limit effort="1" velocity="20" />
     </joint>
     <link name="rolete_22">
@@ -1160,12 +1182,13 @@
         </inertial>
     </link>
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