Commit message: Add full_robot urdf

File: software/src/full_robot/urdf/manipulator.xacro (robot description, xacro)
@@ -4,5 +4,5 @@
 <robot name="manipulator" xmlns:xacro="http://www.ros.org/wiki/xacro">
   <joint name="base_to_link_1" type="fixed">
-    <origin rpy="0 0 -1.57" xyz="0.05 -0.15 0.8"/>
+    <origin rpy="0 0 -1.57" xyz="0.05 -0.15 0.5"/>
     <parent link="base"/>
     <child link="link_1_manip"/>

File: software/src/full_robot/urdf/robot.xacro (robot description, xacro)
@@ -7,7 +7,7 @@
   <link name="base">
     <inertial>
-      <origin xyz="-2.45779e-17 -0.00736431 0.141268" rpy="0 0 0"/>
-      <mass value="9.03432"/>
-      <inertia ixx="0.588684" ixy="-1.30104e-17" ixz="3.46945e-18" iyy="0.584311" iyz="0.0754151" izz="0.304924"/>
+      <origin xyz="7.15175e-09 0.00387039 0.176709" rpy="0 0 0"/>
+      <mass value="14.1165"/>
+      <inertia ixx="0.712488" ixy="-3.32307e-08" ixz="2.04252e-08" iyy="0.743813" iyz="0.0147188" izz="0.588331"/>
     </inertial>
     <!-- Part imu -->
@@ -77,5 +77,5 @@
     <!-- Part mdf_tampa -->
     <visual>
-      <origin xyz="6.93889e-18 -4.16334e-17 0.794" rpy="0 -0 -1.5708"/>
+      <origin xyz="-1.54582e-17 -4.16334e-17 0.4975" rpy="0 -0 -1.5708"/>
       <geometry>
         <mesh filename="file://$(find full_robot)/assets/mdf_tampa.stl"/>
@@ -86,5 +86,5 @@
     </visual>
     <collision>
-      <origin xyz="6.93889e-18 -4.16334e-17 0.794" rpy="0 -0 -1.5708"/>
+      <origin xyz="-1.54582e-17 -4.16334e-17 0.4975" rpy="0 -0 -1.5708"/>
       <geometry>
         <mesh filename="file://$(find full_robot)/assets/mdf_tampa.stl"/>
@@ -98,5 +98,5 @@
       </geometry>
       <material name="capa_baixo_material">
-        <color rgba="0.615686 0.811765 0.929412 1"/>
+        <color rgba="0.901961 0.901961 0.901961 1"/>
       </material>
     </visual>
@@ -178,5 +178,5 @@
       </geometry>
       <material name="capa_cima_material">
-        <color rgba="0.615686 0.811765 0.929412 1"/>
+        <color rgba="0.901961 0.901961 0.901961 1"/>
       </material>
     </visual>
@@ -269,5 +269,5 @@
     <!-- Part perfil_coluna_2 -->
     <visual>
-      <origin xyz="0.17353 -0.100188 0.4" rpy="0 -0 1.0472"/>
+      <origin xyz="0.17353 -0.100188 0.25175" rpy="0 -0 1.0472"/>
       <geometry>
         <mesh filename="file://$(find full_robot)/assets/perfil_coluna__2.stl"/>
@@ -278,5 +278,5 @@
     </visual>
     <collision>
-      <origin xyz="0.17353 -0.100188 0.4" rpy="0 -0 1.0472"/>
+      <origin xyz="0.17353 -0.100188 0.25175" rpy="0 -0 1.0472"/>
       <geometry>
         <mesh filename="file://$(find full_robot)/assets/perfil_coluna__2.stl"/>
@@ -285,5 +285,5 @@
     <!-- Part perfil_coluna_3 -->
     <visual>
-      <origin xyz="-0.17353 -0.100188 0.4" rpy="0 -0 -1.0472"/>
+      <origin xyz="-0.17353 -0.100188 0.25175" rpy="0 -0 -1.0472"/>
       <geometry>
         <mesh filename="file://$(find full_robot)/assets/perfil_coluna__2.stl"/>
@@ -294,5 +294,5 @@
     </visual>
     <collision>
-      <origin xyz="-0.17353 -0.100188 0.4" rpy="0 -0 -1.0472"/>
+      <origin xyz="-0.17353 -0.100188 0.25175" rpy="0 -0 -1.0472"/>
       <geometry>
         <mesh filename="file://$(find full_robot)/assets/perfil_coluna__2.stl"/>
@@ -315,15 +315,111 @@
       </geometry>
     </collision>
+    <!-- Part perfil_coluna_carga -->
+    <visual>
+      <origin xyz="5.01335e-14 4.25077e-14 0.214" rpy="0 -0 -3.14159"/>
+      <geometry>
+        <mesh filename="file://$(find full_robot)/assets/perfil_coluna_carga.stl"/>
+      </geometry>
+      <material name="perfil_coluna_carga_material">
+        <color rgba="0.901961 0.901961 0.901961 1"/>
+      </material>
+    </visual>
+    <collision>
+      <origin xyz="5.01335e-14 4.25077e-14 0.214" rpy="0 -0 -3.14159"/>
+      <geometry>
+        <mesh filename="file://$(find full_robot)/assets/perfil_coluna_carga.stl"/>
+      </geometry>
+    </collision>
+    <!-- Part capa_carga -->
+    <visual>
+      <origin xyz="6.245e-17 9.71445e-17 0.214" rpy="0 -0 -1.5708"/>
+      <geometry>
+        <mesh filename="file://$(find full_robot)/assets/capa_carga.stl"/>
+      </geometry>
+      <material name="capa_carga_material">
+        <color rgba="0.901961 0.901961 0.901961 1"/>
+      </material>
+    </visual>
+    <collision>
+      <origin xyz="6.245e-17 9.71445e-17 0.214" rpy="0 -0 -1.5708"/>
+      <geometry>
+        <mesh filename="file://$(find full_robot)/assets/capa_carga.stl"/>
+      </geometry>
+    </collision>
+    <!-- Part perfil_coluna_carga_2 -->
+    <visual>
+      <origin xyz="6.245e-17 9.71445e-17 0.214" rpy="0 -0 -1.5708"/>
+      <geometry>
+        <mesh filename="file://$(find full_robot)/assets/perfil_coluna_carga.stl"/>
+      </geometry>
+      <material name="perfil_coluna_carga_2_material">
+        <color rgba="0.901961 0.901961 0.901961 1"/>
+      </material>
+    </visual>
+    <collision>
+      <origin xyz="6.245e-17 9.71445e-17 0.214" rpy="0 -0 -1.5708"/>
+      <geometry>
+        <mesh filename="file://$(find full_robot)/assets/perfil_coluna_carga.stl"/>
+      </geometry>
+    </collision>
+    <!-- Part perfil_coluna_carga_3 -->
+    <visual>
+      <origin xyz="0.48 -7.1487e-15 0.214" rpy="0 -0 -1.5708"/>
+      <geometry>
+        <mesh filename="file://$(find full_robot)/assets/perfil_coluna_carga.stl"/>
+      </geometry>
+      <material name="perfil_coluna_carga_3_material">
+        <color rgba="0.901961 0.901961 0.901961 1"/>
+      </material>
+    </visual>
+    <collision>
+      <origin xyz="0.48 -7.1487e-15 0.214" rpy="0 -0 -1.5708"/>
+      <geometry>
+        <mesh filename="file://$(find full_robot)/assets/perfil_coluna_carga.stl"/>
+      </geometry>
+    </collision>
+    <!-- Part mdf_carga -->
+    <visual>
+      <origin xyz="6.245e-17 9.71445e-17 0.4975" rpy="0 -0 -1.5708"/>
+      <geometry>
+        <mesh filename="file://$(find full_robot)/assets/mdf_carga.stl"/>
+      </geometry>
+      <material name="mdf_carga_material">
+        <color rgba="0.901961 0.835294 0.67451 1"/>
+      </material>
+    </visual>
+    <collision>
+      <origin xyz="6.245e-17 9.71445e-17 0.4975" rpy="0 -0 -1.5708"/>
+      <geometry>
+        <mesh filename="file://$(find full_robot)/assets/mdf_carga.stl"/>
+      </geometry>
+    </collision>
+    <!-- Part mdf_carga_2 -->
+    <visual>
+      <origin xyz="6.245e-17 9.71445e-17 0.214" rpy="0 -0 -1.5708"/>
+      <geometry>
+        <mesh filename="file://$(find full_robot)/assets/mdf_carga.stl"/>
+      </geometry>
+      <material name="mdf_carga_2_material">
+        <color rgba="0.901961 0.835294 0.67451 1"/>
+      </material>
+    </visual>
+    <collision>
+      <origin xyz="6.245e-17 9.71445e-17 0.214" rpy="0 -0 -1.5708"/>
+      <geometry>
+        <mesh filename="file://$(find full_robot)/assets/mdf_carga.stl"/>
+      </geometry>
+    </collision>
   </link>
   <!-- Link roda -->
   <link name="roda">
     <inertial>
-      <origin xyz="2.45559e-17 -4.63561e-18 -0.0362488" rpy="0 0 0"/>
+      <origin xyz="2.51575e-17 -5.10809e-18 -0.0362488" rpy="0 0 0"/>
       <mass value="0.174179"/>
-      <inertia ixx="0.000112667" ixy="0" ixz="1.65959e-20" iyy="0.000112667" iyz="0" izz="0.000186298"/>
+      <inertia ixx="0.000112667" ixy="0" ixz="1.92475e-20" iyy="0.000112667" iyz="0" izz="0.000186298"/>
     </inertial>
     <!-- Part roda -->
     <visual>
-      <origin xyz="2.1469e-17 0 -0.038" rpy="1.5708 -5.55112e-17 0"/>
+      <origin xyz="2.2562e-17 0 -0.038" rpy="1.5708 -6.58658e-17 0"/>
       <geometry>
         <mesh filename="file://$(find full_robot)/assets/roda.stl"/>
@@ -334,5 +430,5 @@
     </visual>
     <collision>
-      <origin xyz="2.1469e-17 0 -0.038" rpy="1.5708 -5.55112e-17 0"/>
+      <origin xyz="2.2562e-17 0 -0.038" rpy="1.5708 -6.58658e-17 0"/>
       <geometry>
         <mesh filename="file://$(find full_robot)/assets/roda.stl"/>
@@ -343,7 +439,7 @@
   <link name="rolete">
     <inertial>
-      <origin xyz="1.46499e-50 8.82616e-19 -0.0175" rpy="0 0 0"/>
-      <mass value="0.00952544"/>
-      <inertia ixx="1.03687e-06" ixy="0" ixz="1.15116e-22" iyy="1.03687e-06" iyz="0" izz="4.20254e-07"/>
+      <origin xyz="-1.88278e-33 8.82616e-19 -0.0175" rpy="0 0 0"/>
+      <mass value="0.00952544"/>
+      <inertia ixx="1.03687e-06" ixy="0" ixz="4.88821e-23" iyy="1.03687e-06" iyz="0" izz="4.20254e-07"/>
     </inertial>
     <!-- Part rolete -->
@@ -365,5 +461,5 @@
   </link>
   <!-- Joint from roda to rolete -->
-  <joint name="w1_external_1_passive" type="fixed">
+  <joint name="w1_external_1_passive" type="revolute">
     <origin xyz="0.0175 -0.05 -0.047" rpy="-3.14159 -1.5708 0"/>
     <parent link="roda"/>
@@ -375,11 +471,11 @@
   <link name="rolete_2">
     <inertial>
-      <origin xyz="1.38778e-17 1.52538e-20 -0.0175" rpy="0 0 0"/>
-      <mass value="0.00952544"/>
-      <inertia ixx="1.03687e-06" ixy="-1.27301e-22" ixz="-2.33288e-23" iyy="1.03687e-06" iyz="-1.63191e-23" izz="4.20254e-07"/>
+      <origin xyz="2.42861e-17 1.52538e-20 -0.0175" rpy="0 0 0"/>
+      <mass value="0.00952544"/>
+      <inertia ixx="1.03687e-06" ixy="-9.85217e-23" ixz="4.55279e-23" iyy="1.03687e-06" iyz="1.27078e-23" izz="4.20254e-07"/>
     </inertial>
     <!-- Part rolete_2 -->
     <visual>
-      <origin xyz="1.38778e-17 0 -0.0175" rpy="1.5708 1.5708 0"/>
+      <origin xyz="2.42861e-17 0 -0.0175" rpy="1.5708 1.5708 0"/>
       <geometry>
         <mesh filename="file://$(find full_robot)/assets/rolete.stl"/>
@@ -390,5 +486,5 @@
     </visual>
     <collision>
-      <origin xyz="1.38778e-17 0 -0.0175" rpy="1.5708 1.5708 0"/>
+      <origin xyz="2.42861e-17 0 -0.0175" rpy="1.5708 1.5708 0"/>
       <geometry>
         <mesh filename="file://$(find full_robot)/assets/rolete.stl"/>
@@ -397,6 +493,6 @@
   </link>
   <!-- Joint from roda to rolete_2 -->
-  <joint name="w1_external_2_passive" type="fixed">
-    <origin xyz="0.0520513 -0.00984456 -0.047" rpy="1.5708 5.55112e-17 2.61799"/>
+  <joint name="w1_external_2_passive" type="revolute">
+    <origin xyz="0.0520513 -0.00984456 -0.047" rpy="1.5708 4.16334e-17 2.61799"/>
     <parent link="roda"/>
     <child link="rolete_2"/>
@@ -407,11 +503,11 @@
   <link name="rolete_3">
     <inertial>
-      <origin xyz="-5.55112e-17 -5.54959e-17 -0.0175" rpy="0 0 0"/>
-      <mass value="0.00952544"/>
-      <inertia ixx="1.03687e-06" ixy="-8.46859e-23" ixz="-8.08867e-23" iyy="1.03687e-06" iyz="-3.46581e-23" izz="4.20254e-07"/>
+      <origin xyz="-5.55112e-17 1.52538e-20 -0.0175" rpy="0 0 0"/>
+      <mass value="0.00952544"/>
+      <inertia ixx="1.03687e-06" ixy="-1.13465e-22" ixz="-4.91065e-23" iyy="1.03687e-06" iyz="-4.74348e-23" izz="4.20254e-07"/>
     </inertial>
     <!-- Part rolete_3 -->
     <visual>
-      <origin xyz="-5.55112e-17 -5.55112e-17 -0.0175" rpy="1.5708 1.5708 0"/>
+      <origin xyz="-5.55112e-17 0 -0.0175" rpy="1.5708 1.5708 0"/>
       <geometry>
         <mesh filename="file://$(find full_robot)/assets/rolete.stl"/>
@@ -422,5 +518,5 @@
     </visual>
     <collision>
-      <origin xyz="-5.55112e-17 -5.55112e-17 -0.0175" rpy="1.5708 1.5708 0"/>
+      <origin xyz="-5.55112e-17 0 -0.0175" rpy="1.5708 1.5708 0"/>
       <geometry>
         <mesh filename="file://$(find full_robot)/assets/rolete.stl"/>
@@ -429,6 +525,6 @@
   </link>
   <!-- Joint from roda to rolete_3 -->
-  <joint name="w1_external_3_passive" type="fixed">
-    <origin xyz="0.0520513 0.00984456 -0.047" rpy="-1.5708 5.55112e-17 -2.61799"/>
+  <joint name="w1_external_3_passive" type="revolute">
+    <origin xyz="0.0520513 0.00984456 -0.047" rpy="-1.5708 4.16334e-17 -2.61799"/>
     <parent link="roda"/>
     <child link="rolete_3"/>
@@ -439,7 +535,7 @@
   <link name="rolete_4">
     <inertial>
-      <origin xyz="1.46499e-50 1.52538e-20 -0.0175" rpy="0 0 0"/>
-      <mass value="0.00952544"/>
-      <inertia ixx="1.03687e-06" ixy="0" ixz="1.15116e-22" iyy="1.03687e-06" iyz="0" izz="4.20254e-07"/>
+      <origin xyz="-1.88278e-33 1.52538e-20 -0.0175" rpy="0 0 0"/>
+      <mass value="0.00952544"/>
+      <inertia ixx="1.03687e-06" ixy="0" ixz="4.88821e-23" iyy="1.03687e-06" iyz="0" izz="4.20254e-07"/>
     </inertial>
     <!-- Part rolete_4 -->
@@ -461,5 +557,5 @@
   </link>
   <!-- Joint from roda to rolete_4 -->
-  <joint name="w1_external_4_passive" type="fixed">
+  <joint name="w1_external_4_passive" type="revolute">
     <origin xyz="0.0175 0.05 -0.047" rpy="-3.14159 -1.5708 0"/>
     <parent link="roda"/>
@@ -471,11 +567,11 @@
   <link name="rolete_5">
     <inertial>
-      <origin xyz="1.38778e-17 -5.54959e-17 -0.0175" rpy="0 0 0"/>
-      <mass value="0.00952544"/>
-      <inertia ixx="1.03687e-06" ixy="-4.09638e-23" ixz="-4.61173e-40" iyy="1.03687e-06" iyz="-2.8816e-23" izz="4.20254e-07"/>
+      <origin xyz="2.77556e-17 -5.54959e-17 -0.0175" rpy="0 0 0"/>
+      <mass value="0.00952544"/>
+      <inertia ixx="1.03687e-06" ixy="-4.09638e-23" ixz="-1.08183e-23" iyy="1.03687e-06" iyz="-6.5886e-23" izz="4.20254e-07"/>
     </inertial>
     <!-- Part rolete_5 -->
     <visual>
-      <origin xyz="1.38778e-17 -5.55112e-17 -0.0175" rpy="1.5708 1.5708 0"/>
+      <origin xyz="2.77556e-17 -5.55112e-17 -0.0175" rpy="1.5708 1.5708 0"/>
       <geometry>
         <mesh filename="file://$(find full_robot)/assets/rolete.stl"/>
@@ -486,5 +582,5 @@
     </visual>
     <collision>
-      <origin xyz="1.38778e-17 -5.55112e-17 -0.0175" rpy="1.5708 1.5708 0"/>
+      <origin xyz="2.77556e-17 -5.55112e-17 -0.0175" rpy="1.5708 1.5708 0"/>
       <geometry>
         <mesh filename="file://$(find full_robot)/assets/rolete.stl"/>
@@ -493,6 +589,6 @@
   </link>
   <!-- Joint from roda to rolete_5 -->
-  <joint name="w1_external_5_passive" type="fixed">
-    <origin xyz="-0.0345513 0.0401554 -0.047" rpy="1.5708 1.11022e-16 2.61799"/>
+  <joint name="w1_external_5_passive" type="revolute">
+    <origin xyz="-0.0345513 0.0401554 -0.047" rpy="1.5708 9.71445e-17 2.61799"/>
     <parent link="roda"/>
     <child link="rolete_5"/>
@@ -503,11 +599,11 @@
   <link name="rolete_6">
     <inertial>
-      <origin xyz="-1.38778e-17 1.52538e-20 -0.0175" rpy="0 0 0"/>
-      <mass value="0.00952544"/>
-      <inertia ixx="1.03687e-06" ixy="2.85021e-23" ixz="-4.66576e-23" iyy="1.03687e-06" iyz="7.23183e-24" izz="4.20254e-07"/>
+      <origin xyz="-1.04083e-17 1.52538e-20 -0.0175" rpy="0 0 0"/>
+      <mass value="0.00952544"/>
+      <inertia ixx="1.03687e-06" ixy="-2.76823e-25" ixz="5.07067e-23" iyy="1.03687e-06" iyz="6.9839e-24" izz="4.20254e-07"/>
     </inertial>
     <!-- Part rolete_6 -->
     <visual>
-      <origin xyz="-1.38778e-17 0 -0.0175" rpy="1.5708 1.5708 0"/>
+      <origin xyz="-1.04083e-17 0 -0.0175" rpy="1.5708 1.5708 0"/>
       <geometry>
         <mesh filename="file://$(find full_robot)/assets/rolete.stl"/>
@@ -518,5 +614,5 @@
     </visual>
     <collision>
-      <origin xyz="-1.38778e-17 0 -0.0175" rpy="1.5708 1.5708 0"/>
+      <origin xyz="-1.04083e-17 0 -0.0175" rpy="1.5708 1.5708 0"/>
       <geometry>
         <mesh filename="file://$(find full_robot)/assets/rolete.stl"/>
@@ -525,6 +621,6 @@
   </link>
   <!-- Joint from roda to rolete_6 -->
-  <joint name="w1_external_6_passive" type="fixed">
-    <origin xyz="-0.0345513 -0.0401554 -0.047" rpy="-1.5708 5.55112e-17 -2.61799"/>
+  <joint name="w1_external_6_passive" type="revolute">
+    <origin xyz="-0.0345513 -0.0401554 -0.047" rpy="-1.5708 4.16334e-17 -2.61799"/>
     <parent link="roda"/>
     <child link="rolete_6"/>
@@ -535,11 +631,11 @@
   <link name="rolete_7">
     <inertial>
-      <origin xyz="-1.06152e-32 -1.03931e-17 -0.0175" rpy="0 0 0"/>
-      <mass value="0.00952544"/>
-      <inertia ixx="1.03687e-06" ixy="1.87444e-37" ixz="7.67209e-23" iyy="1.03687e-06" iyz="4.66576e-23" izz="4.20254e-07"/>
+      <origin xyz="-2.77556e-17 6.95415e-18 -0.0175" rpy="0 0 0"/>
+      <mass value="0.00952544"/>
+      <inertia ixx="1.03687e-06" ixy="-9.19819e-23" ixz="-7.59568e-23" iyy="1.03687e-06" iyz="-3.2944e-23" izz="4.20254e-07"/>
     </inertial>
     <!-- Part rolete_7 -->
     <visual>
-      <origin xyz="0 -1.04083e-17 -0.0175" rpy="1.5708 1.5708 0"/>
+      <origin xyz="-2.77556e-17 6.93889e-18 -0.0175" rpy="1.5708 1.5708 0"/>
       <geometry>
         <mesh filename="file://$(find full_robot)/assets/rolete.stl"/>
@@ -550,5 +646,5 @@
     </visual>
     <collision>
-      <origin xyz="0 -1.04083e-17 -0.0175" rpy="1.5708 1.5708 0"/>
+      <origin xyz="-2.77556e-17 6.93889e-18 -0.0175" rpy="1.5708 1.5708 0"/>
       <geometry>
         <mesh filename="file://$(find full_robot)/assets/rolete.stl"/>
@@ -557,5 +653,5 @@
   </link>
   <!-- Joint from roda to rolete_7 -->
-  <joint name="w1_internal_1_passive" type="fixed">
+  <joint name="w1_internal_1_passive" type="revolute">
     <origin xyz="0.00984456 -0.0520513 -0.029" rpy="0.523599 -1.5708 0"/>
     <parent link="roda"/>
@@ -567,11 +663,11 @@
   <link name="rolete_8">
     <inertial>
-      <origin xyz="6.93889e-18 -2.77403e-17 -0.0175" rpy="0 0 0"/>
-      <mass value="0.00952544"/>
-      <inertia ixx="1.03687e-06" ixy="-1.15116e-22" ixz="0" iyy="1.03687e-06" iyz="0" izz="4.20254e-07"/>
+      <origin xyz="-1.38778e-17 -2.77403e-17 -0.0175" rpy="0 0 0"/>
+      <mass value="0.00952544"/>
+      <inertia ixx="1.03687e-06" ixy="-1.53672e-22" ixz="0" iyy="1.03687e-06" iyz="0" izz="4.20254e-07"/>
     </inertial>
     <!-- Part rolete_8 -->
     <visual>
-      <origin xyz="6.93889e-18 -2.77556e-17 -0.0175" rpy="1.5708 1.5708 0"/>
+      <origin xyz="-1.38778e-17 -2.77556e-17 -0.0175" rpy="1.5708 1.5708 0"/>
       <geometry>
         <mesh filename="file://$(find full_robot)/assets/rolete.stl"/>
@@ -582,5 +678,5 @@
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