Commit message: URDF with write colors

File: software/src/full_robot/urdf/manipulator.xacro (robot description, xacro)
@@ -4,5 +4,5 @@
 <robot name="manipulator" xmlns:xacro="http://www.ros.org/wiki/xacro">
   <joint name="base_to_link_1" type="fixed">
-    <origin rpy="0 0 -1.57" xyz="0.05 -0.15 0.5"/>
+    <origin rpy="0 0 -1.57" xyz="0.05 -0.15 0.505"/>
     <parent link="base"/>
     <child link="link_1_manip"/>

File: software/src/full_robot/urdf/robot.xacro (robot description, xacro)
@@ -4,5 +4,4 @@
 <robot name="my-robot" xmlns:xacro="http://www.ros.org/wiki/xacro">
   <xacro:include filename="$(find full_robot)/urdf/manipulator.xacro"/>
-  <!-- Link base -->
   <link name="base">
     <inertial>
@@ -11,7 +10,8 @@
       <inertia ixx="0.712488" ixy="-3.32307e-08" ixz="2.04252e-08" iyy="0.743813" iyz="0.0147188" izz="0.588331"/>
     </inertial>
-    <!-- Part imu -->
-    <visual>
-      <origin xyz="-2.36447e-17 -5.80614e-17 0.083" rpy="0 -0 6.12323e-17"/>
+  </link>
+  <link name="imu_link">
+    <visual>
+      <origin xyz="0 0 0" rpy="0 0 0"/>
       <geometry>
         <mesh filename="file://$(find full_robot)/assets/imu.stl"/>
@@ -22,12 +22,18 @@
     </visual>
     <collision>
-      <origin xyz="-2.36447e-17 -5.80614e-17 0.083" rpy="0 -0 6.12323e-17"/>
+      <origin xyz="0 0 0" rpy="0 0 0"/>
       <geometry>
         <mesh filename="file://$(find full_robot)/assets/imu.stl"/>
       </geometry>
     </collision>
-    <!-- Part lidar -->
-    <visual>
-      <origin xyz="-2.24826e-17 -6.22208e-17 0.092" rpy="0 -0 6.12323e-17"/>
+  </link>
+  <joint name="base_to_imu" type="fixed">
+    <parent link="base"/>
+    <child link="imu_link"/>
+    <origin xyz="-2.36447e-17 -5.80614e-17 0.083" rpy="0 0 6.12323e-17"/>
+  </joint>
+  <link name="lidar_link">
+    <visual>
+      <origin xyz="0 0 0" rpy="0 0 0"/>
       <geometry>
         <mesh filename="file://$(find full_robot)/assets/lidar.stl"/>
@@ -38,12 +44,18 @@
     </visual>
     <collision>
-      <origin xyz="-2.24826e-17 -6.22208e-17 0.092" rpy="0 -0 6.12323e-17"/>
+      <origin xyz="0 0 0" rpy="0 0 0"/>
       <geometry>
         <mesh filename="file://$(find full_robot)/assets/lidar.stl"/>
       </geometry>
     </collision>
-    <!-- Part motor -->
-    <visual>
-      <origin xyz="0 0.155075 -0.04535" rpy="0 -0 -3.14159"/>
+  </link>
+  <joint name="base_to_lidar" type="fixed">
+    <parent link="base"/>
+    <child link="lidar_link"/>
+    <origin xyz="-2.24826e-17 -6.22208e-17 0.092" rpy="0 0 6.12323e-17"/>
+  </joint>
+  <link name="motor_link">
+    <visual>
+      <origin xyz="0 0 0" rpy="0 0 0"/>
       <geometry>
         <mesh filename="file://$(find full_robot)/assets/motor.stl"/>
@@ -54,44 +66,62 @@
     </visual>
     <collision>
-      <origin xyz="0 0.155075 -0.04535" rpy="0 -0 -3.14159"/>
+      <origin xyz="0 0 0" rpy="0 0 0"/>
       <geometry>
         <mesh filename="file://$(find full_robot)/assets/motor.stl"/>
       </geometry>
     </collision>
-    <!-- Part mdf_motores -->
-    <visual>
-      <origin xyz="0 0 0" rpy="0 -0 -1.5708"/>
+  </link>
+  <joint name="base_to_motor" type="fixed">
+    <parent link="base"/>
+    <child link="motor_link"/>
+    <origin xyz="0 0.155075 -0.04535" rpy="0 0 -3.14159"/>
+  </joint>
+  <link name="mdf_motores_link">
+    <visual>
+      <origin xyz="0 0 0" rpy="0 0 0"/>
       <geometry>
         <mesh filename="file://$(find full_robot)/assets/mdf_motores.stl"/>
       </geometry>
       <material name="mdf_motores_material">
-        <color rgba="0.901961 0.835294 0.67451 1"/>
-      </material>
-    </visual>
-    <collision>
-      <origin xyz="0 0 0" rpy="0 -0 -1.5708"/>
+        <color rgba="0.84 0.78 0.63 1.0"/>
+      </material>
+    </visual>
+    <collision>
+      <origin xyz="0 0 0" rpy="0 0 0"/>
       <geometry>
         <mesh filename="file://$(find full_robot)/assets/mdf_motores.stl"/>
       </geometry>
     </collision>
-    <!-- Part mdf_tampa -->
-    <visual>
-      <origin xyz="-1.54582e-17 -4.16334e-17 0.4975" rpy="0 -0 -1.5708"/>
+  </link>
+  <joint name="base_to_mdf_motores" type="fixed">
+    <parent link="base"/>
+    <child link="mdf_motores_link"/>
+    <origin xyz="0 0 0" rpy="0 0 -1.5708"/>
+  </joint>
+  <link name="mdf_tampa_link">
+    <visual>
+      <origin xyz="0 0 0" rpy="0 0 0"/>
       <geometry>
         <mesh filename="file://$(find full_robot)/assets/mdf_tampa.stl"/>
       </geometry>
       <material name="mdf_tampa_material">
-        <color rgba="0.901961 0.835294 0.67451 1"/>
-      </material>
-    </visual>
-    <collision>
-      <origin xyz="-1.54582e-17 -4.16334e-17 0.4975" rpy="0 -0 -1.5708"/>
+        <color rgba="0.84 0.78 0.63 1.0"/>
+      </material>
+    </visual>
+    <collision>
+      <origin xyz="0 0 0" rpy="0 0 0"/>
       <geometry>
         <mesh filename="file://$(find full_robot)/assets/mdf_tampa.stl"/>
       </geometry>
     </collision>
-    <!-- Part capa_baixo -->
-    <visual>
-      <origin xyz="6.93889e-18 -4.16334e-17 -0.078" rpy="0 -0 6.12323e-17"/>
+  </link>
+  <joint name="base_to_mdf_tampa" type="fixed">
+    <parent link="base"/>
+    <child link="mdf_tampa_link"/>
+    <origin xyz="-1.54582e-17 -4.16334e-17 0.4975" rpy="0 0 -1.5708"/>
+  </joint>
+  <link name="capa_baixo_link">
+    <visual>
+      <origin xyz="0 0 0" rpy="0 0 0"/>
       <geometry>
         <mesh filename="file://$(find full_robot)/assets/capa_baixo.stl"/>
@@ -102,44 +132,62 @@
     </visual>
     <collision>
-      <origin xyz="6.93889e-18 -4.16334e-17 -0.078" rpy="0 -0 6.12323e-17"/>
+      <origin xyz="0 0 0" rpy="0 0 0"/>
       <geometry>
         <mesh filename="file://$(find full_robot)/assets/capa_baixo.stl"/>
       </geometry>
     </collision>
-    <!-- Part mdf -->
-    <visual>
-      <origin xyz="1.54074e-33 -1.38778e-17 0.086" rpy="0 -0 -1.5708"/>
+  </link>
+  <joint name="base_to_capa_baixo" type="fixed">
+    <parent link="base"/>
+    <child link="capa_baixo_link"/>
+    <origin xyz="6.93889e-18 -4.16334e-17 -0.078" rpy="0 0 0"/>
+  </joint>
+  <link name="mdf_link">
+    <visual>
+      <origin xyz="0 0 0" rpy="0 0 0"/>
       <geometry>
         <mesh filename="file://$(find full_robot)/assets/mdf.stl"/>
       </geometry>
       <material name="mdf_material">
-        <color rgba="0.901961 0.835294 0.67451 1"/>
-      </material>
-    </visual>
-    <collision>
-      <origin xyz="1.54074e-33 -1.38778e-17 0.086" rpy="0 -0 -1.5708"/>
+        <color rgba="0.84 0.78 0.63 1.0"/>
+      </material>
+    </visual>
+    <collision>
+      <origin xyz="0 0 0" rpy="0 0 0"/>
       <geometry>
         <mesh filename="file://$(find full_robot)/assets/mdf.stl"/>
       </geometry>
     </collision>
-    <!-- Part mdf_2 -->
-    <visual>
-      <origin xyz="1.54074e-33 -1.38778e-17 0.132" rpy="0 -0 -1.5708"/>
+  </link>
+  <joint name="base_to_mdf" type="fixed">
+    <parent link="base"/>
+    <child link="mdf_link"/>
+    <origin xyz="1.54074e-33 -1.38778e-17 0.086" rpy="0 0 -1.5708"/>
+  </joint>
+  <link name="mdf_2_link">
+    <visual>
+      <origin xyz="0 0 0" rpy="0 0 0"/>
       <geometry>
         <mesh filename="file://$(find full_robot)/assets/mdf.stl"/>
       </geometry>
       <material name="mdf_2_material">
-        <color rgba="0.901961 0.835294 0.67451 1"/>
-      </material>
-    </visual>
-    <collision>
-      <origin xyz="1.54074e-33 -1.38778e-17 0.132" rpy="0 -0 -1.5708"/>
+        <color rgba="0.84 0.78 0.63 1.0"/>
+      </material>
+    </visual>
+    <collision>
+      <origin xyz="0 0 0" rpy="0 0 0"/>
       <geometry>
         <mesh filename="file://$(find full_robot)/assets/mdf.stl"/>
       </geometry>
     </collision>
-    <!-- Part led -->
-    <visual>
-      <origin xyz="6.93889e-18 -4.16334e-17 0.142" rpy="0 -0 6.12323e-17"/>
+  </link>
+  <joint name="base_to_mdf_2" type="fixed">
+    <parent link="base"/>
+    <child link="mdf_2_link"/>
+    <origin xyz="1.54074e-33 -1.38778e-17 0.132" rpy="0 0 -1.5708"/>
+  </joint>
+  <link name="led_link">
+    <visual>
+      <origin xyz="0 0 0" rpy="0 0 0"/>
       <geometry>
         <mesh filename="file://$(find full_robot)/assets/led.stl"/>
@@ -150,12 +198,18 @@
     </visual>
     <collision>
-      <origin xyz="6.93889e-18 -4.16334e-17 0.142" rpy="0 -0 6.12323e-17"/>
+      <origin xyz="0 0 0" rpy="0 0 0"/>
       <geometry>
         <mesh filename="file://$(find full_robot)/assets/led.stl"/>
       </geometry>
     </collision>
-    <!-- Part perfil_motores -->
-    <visual>
-      <origin xyz="0 0.207375 -0.01" rpy="0 -0 -3.14159"/>
+  </link>
+  <joint name="base_to_led" type="fixed">
+    <parent link="base"/>
+    <child link="led_link"/>
+    <origin xyz="6.93889e-18 -4.16334e-17 0.142" rpy="0 0 0"/>
+  </joint>
+  <link name="perfil_motores_link">
+    <visual>
+      <origin xyz="0 0 0" rpy="0 0 0"/>
       <geometry>
         <mesh filename="file://$(find full_robot)/assets/perfil_motores.stl"/>
@@ -166,12 +220,18 @@
     </visual>
     <collision>
-      <origin xyz="0 0.207375 -0.01" rpy="0 -0 -3.14159"/>
+      <origin xyz="0 0 0" rpy="0 0 0"/>
       <geometry>
         <mesh filename="file://$(find full_robot)/assets/perfil_motores.stl"/>
       </geometry>
     </collision>
-    <!-- Part capa_cima -->
-    <visual>
-      <origin xyz="6.93889e-18 -4.16334e-17 0.142" rpy="0 -0 6.12323e-17"/>
+  </link>
+  <joint name="base_to_perfil_motores" type="fixed">
+    <parent link="base"/>
+    <child link="perfil_motores_link"/>
+    <origin xyz="0 0.207375 -0.01" rpy="0 0 -3.14159"/>
+  </joint>
+  <link name="capa_cima_link">
+    <visual>
+      <origin xyz="0 0 0" rpy="0 0 0"/>
       <geometry>
         <mesh filename="file://$(find full_robot)/assets/capa_cima.stl"/>
@@ -182,12 +242,18 @@
     </visual>
     <collision>
-      <origin xyz="6.93889e-18 -4.16334e-17 0.142" rpy="0 -0 6.12323e-17"/>
+      <origin xyz="0 0 0" rpy="0 0 0"/>
       <geometry>
         <mesh filename="file://$(find full_robot)/assets/capa_cima.stl"/>
       </geometry>
     </collision>
-    <!-- Part perfil_coluna -->
-    <visual>
-      <origin xyz="1.92083e-17 0.200375 0.107" rpy="0 -0 2.10573e-16"/>
+  </link>
+  <joint name="base_to_capa_cima" type="fixed">
+    <parent link="base"/>
+    <child link="capa_cima_link"/>
+    <origin xyz="6.93889e-18 -4.16334e-17 0.142" rpy="0 0 0"/>
+  </joint>
+  <link name="perfil_coluna_link">
+    <visual>
+      <origin xyz="0 0 0" rpy="0 0 0"/>
       <geometry>
         <mesh filename="file://$(find full_robot)/assets/perfil_coluna.stl"/>
@@ -198,12 +264,18 @@
     </visual>
     <collision>
-      <origin xyz="1.92083e-17 0.200375 0.107" rpy="0 -0 2.10573e-16"/>
+      <origin xyz="0 0 0" rpy="0 0 0"/>
       <geometry>
         <mesh filename="file://$(find full_robot)/assets/perfil_coluna.stl"/>
       </geometry>
     </collision>
-    <!-- Part perfil_motores_2 -->
-    <visual>
-      <origin xyz="-0.179592 -0.103688 -0.01" rpy="0 -0 -1.0472"/>
+  </link>
+  <joint name="base_to_perfil_coluna" type="fixed">
+    <parent link="base"/>
+    <child link="perfil_coluna_link"/>
+    <origin xyz="1.92083e-17 0.200375 0.107" rpy="0 0 0"/>
+  </joint>
+  <link name="perfil_motores_2_link">
+    <visual>
+      <origin xyz="0 0 0" rpy="0 0 0"/>
       <geometry>
         <mesh filename="file://$(find full_robot)/assets/perfil_motores.stl"/>
@@ -214,28 +286,40 @@
     </visual>
     <collision>
-      <origin xyz="-0.179592 -0.103688 -0.01" rpy="0 -0 -1.0472"/>
+      <origin xyz="0 0 0" rpy="0 0 0"/>
       <geometry>
         <mesh filename="file://$(find full_robot)/assets/perfil_motores.stl"/>
       </geometry>
     </collision>
-    <!-- Part mdf_3 -->
-    <visual>
-      <origin xyz="1.54074e-33 -1.38778e-17 0.208" rpy="0 -0 -1.5708"/>
+  </link>
+  <joint name="base_to_perfil_motores_2" type="fixed">
+    <parent link="base"/>
+    <child link="perfil_motores_2_link"/>
+    <origin xyz="-0.179592 -0.103688 -0.01" rpy="0 0 -1.0472"/>
+  </joint>
+  <link name="mdf_3_link">
+    <visual>
+      <origin xyz="0 0 0" rpy="0 0 0"/>
       <geometry>
         <mesh filename="file://$(find full_robot)/assets/mdf.stl"/>
       </geometry>
       <material name="mdf_3_material">
-        <color rgba="0.901961 0.835294 0.67451 1"/>
-      </material>
-    </visual>
-    <collision>
-      <origin xyz="1.54074e-33 -1.38778e-17 0.208" rpy="0 -0 -1.5708"/>
+        <color rgba="0.84 0.78 0.63 1.0"/>
+      </material>
+    </visual>
+    <collision>
+      <origin xyz="0 0 0" rpy="0 0 0"/>
       <geometry>
         <mesh filename="file://$(find full_robot)/assets/mdf.stl"/>
       </geometry>
     </collision>
-    <!-- Part motor_2 -->
-    <visual>
-      <origin xyz="0.134299 -0.0775375 -0.04535" rpy="0 -0 1.0472"/>
+  </link>
+  <joint name="base_to_mdf_3" type="fixed">
+    <parent link="base"/>
+    <child link="mdf_3_link"/>
+    <origin xyz="1.54074e-33 -1.38778e-17 0.208" rpy="0 0 -1.5708"/>
+  </joint>
+  <link name="motor_2_link">
+    <visual>
+      <origin xyz="0 0 0" rpy="0 0 0"/>
       <geometry>
         <mesh filename="file://$(find full_robot)/assets/motor.stl"/>
@@ -246,12 +330,18 @@
     </visual>
     <collision>
-      <origin xyz="0.134299 -0.0775375 -0.04535" rpy="0 -0 1.0472"/>
+      <origin xyz="0 0 0" rpy="0 0 0"/>
       <geometry>
         <mesh filename="file://$(find full_robot)/assets/motor.stl"/>
       </geometry>
     </collision>
-    <!-- Part motor_3 -->
-    <visual>
-      <origin xyz="-0.134299 -0.0775375 -0.04535" rpy="0 -0 -1.0472"/>
+  </link>
+  <joint name="base_to_motor_2" type="fixed">
+    <parent link="base"/>
+    <child link="motor_2_link"/>
+    <origin xyz="0.134299 -0.0775375 -0.04535" rpy="0 0 1.0472"/>
+  </joint>
+  <link name="motor_3_link">
+    <visual>
+      <origin xyz="0 0 0" rpy="0 0 0"/>
       <geometry>
         <mesh filename="file://$(find full_robot)/assets/motor.stl"/>
@@ -262,12 +352,18 @@
     </visual>
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